Commit message: AI 待修改 雷达的数据严重漂移

File: ros_ws/src/photo_nav_description/urdf/photo_nav_robot.urdf.xacro (robot description, xacro)
@@ -287,4 +287,36 @@
     </plugin>
   </gazebo>
+  <!-- ==================== IMU SENSOR ==================== -->
+  <link name="imu_link">
+    <inertial>
+      <mass value="0.01"/>
+      <inertia ixx="0.00001" ixy="0" ixz="0" iyy="0.00001" iyz="0" izz="0.00001"/>
+    </inertial>
+  </link>
+  <joint name="imu_joint" type="fixed">
+    <parent link="base_link"/>
+    <child  link="imu_link"/>
+    <origin xyz="0 0 0" rpy="0 0 0"/>
+  </joint>
+  <gazebo reference="imu_link">
+    <sensor name="imu" type="imu">
+      <topic>imu</topic>
+      <ignition_frame_id>imu_link</ignition_frame_id>
+      <update_rate>100</update_rate>
+      <always_on>true</always_on>
+      <imu>
+        <angular_velocity>
+          <x><noise type="gaussian"><mean>0</mean><stddev>0.009</stddev></noise></x>
+          <y><noise type="gaussian"><mean>0</mean><stddev>0.009</stddev></noise></y>
+          <z><noise type="gaussian"><mean>0</mean><stddev>0.009</stddev></noise></z>
+        </angular_velocity>
+        <linear_acceleration>
+          <x><noise type="gaussian"><mean>0</mean><stddev>0.021</stddev></noise></x>
+          <y><noise type="gaussian"><mean>0</mean><stddev>0.021</stddev></noise></y>
+          <z><noise type="gaussian"><mean>0</mean><stddev>0.021</stddev></noise></z>
+        </linear_acceleration>
+      </imu>
+    </sensor>
+  </gazebo>
   <!-- Caster friction override in Gazebo -->
   <gazebo reference="front_caster_link">

Commit message: 主机测试完备

File: ros_ws/src/photo_nav_description/urdf/photo_nav_robot.urdf.xacro (robot description, xacro)
@@ -165,5 +165,5 @@
     z offset from base_link: lidar_z_from_ground - chassis_z
   -->
-  <link name="lidar_link">
+  <link name="laser">
     <visual>
       <origin xyz="0 0 0" rpy="0 0 0"/>
@@ -186,6 +186,5 @@
   <joint name="lidar_joint" type="fixed">
     <parent link="base_link"/>
-    <child  link="lidar_link"/>
-    <!-- On the front face of chassis, 1.0m above ground -->
+    <child  link="laser"/>
     <origin xyz="${chassis_radius} 0 ${lidar_z_from_ground - chassis_z}" rpy="0 0 0"/>
   </joint>
@@ -228,5 +227,5 @@
   </joint>
   <!-- ==================== LIDAR SENSOR PLUGIN ==================== -->
-  <gazebo reference="lidar_link">
+  <gazebo reference="laser">
     <sensor name="lidar" type="gpu_lidar">
       <topic>scan</topic>
